Commit message: Autoware Vehicle Folder

File: vehicle/beliv_sim_launch/beliv_sim_description/urdf/vehicle.xacro (robot description, xacro)
@@ -2,5 +2,5 @@
 <robot xmlns:xacro="http://ros.org/wiki/xacro">
   <!-- load parameter -->
-  <xacro:property name="vehicle_info" value="${load_yaml('$(find beliv_vehicle_description)/config/vehicle_info.param.yaml')}"/>
+  <xacro:property name="vehicle_info" value="${load_yaml('$(find beliv_sim_description)/config/vehicle_info.param.yaml')}"/>
   <!-- vehicle body -->
   <link name="base_link">
@@ -8,5 +8,5 @@
       <origin xyz="${vehicle_info['/**']['ros__parameters']['wheel_base']/2.0} 0 0" rpy="${pi/2.0} 0 ${pi}"/>
       <geometry>
-        <mesh filename="package://beliv_vehicle_description/mesh/mache.dae" scale="1 1 1"/>
+        <mesh filename="package://beliv_sim_description/mesh/mache.dae" scale="1 1 1"/>
       </geometry>
     </visual>
